File: PCB/keyboard.kicad_pcb (KiCad board)
At the start: 2 copper layers, 126 parts, among them SW1 SW_Push, SW10 SW_Push, SW11 SW_Push, SW12 SW_Push, SW13 SW_Push, SW14 SW_Push, SW15 SW_Push, SW16 SW_Push, SW17 SW_Push, SW18 SW_Push, SW19 SW_Push, SW2 SW_Push, SW20 SW_Push, SW21 SW_Push, SW22 SW_Push, SW23 SW_Push, SW24 SW_Push, SW25 SW_Push, SW26 SW_Push, SW27 SW_Push, SW28 SW_Push, SW29 SW_Push, SW3 SW_Push, SW30 SW_Push, SW31 SW_Push, SW32 SW_Push, SW33 SW_Push, SW34 SW_Push, SW35 SW_Push, SW36 SW_Push, SW37 SW_Push, SW38 SW_Push, SW39 SW_Push, SW4 SW_Push, SW40 SW_Push, SW41 SW_Push, SW42 SW_Push, SW43 SW_Push, SW44 SW_Push, SW45 SW_Push, SW46 SW_Push, SW47 SW_Push, SW48 SW_Push, SW49 SW_Push, SW5 SW_Push, SW50 SW_Push, SW51 SW_Push, SW52 SW_Push, SW53 SW_Push, SW54 SW_Push, SW55 SW_Push, SW56 SW_Push, SW57 SW_Push, SW58 SW_Push, SW59 SW_Push, SW6 SW_Push, SW60 SW_Push, SW61 SW_Push, SW62 RotaryEncoder_Switch, SW63 RotaryEncoder_Switch, SW7 SW_Push, SW8 SW_Push, SW9 SW_Push

Commit message: oeiaiaiaoio
Parts:
- added U1: Pico, Module:RaspberryPi_Pico_Common_THT, F.Cu at (16.0, 41.0)
- moved D54 439.6 mm to (14.4, 133.8), turned to 90 degrees
- moved D42 429.9 mm to (14.7, 114.7), turned to 90 degrees
- moved D29 421.5 mm to (14.4, 95.7), turned to 90 degrees
- moved D55 416.3 mm to (37.9, 133.8), turned to 90 degrees
- moved D15 413.2 mm to (14.4, 76.7), turned to 90 degrees
- moved D1 405.6 mm to (14.4, 57.6), turned to 90 degrees
- moved D56 392.4 mm to (61.9, 133.8), turned to 90 degrees
- moved D30 389.2 mm to (47.5, 95.7), turned to 90 degrees
- moved D2 387.8 mm to (33.5, 57.6), turned to 90 degrees
- moved D43 387.5 mm to (57.5, 114.7), turned to 90 degrees
- moved D16 385.6 mm to (43.1, 76.7), turned to 90 degrees
- moved D31 370.9 mm to (66.7, 95.7), turned to 90 degrees
- moved D3 370.4 mm to (52.3, 57.6), turned to 90 degrees
- moved D44 368.9 mm to (76.7, 114.7), turned to 90 degrees
- moved D57 368.6 mm to (86.0, 133.8), turned to 90 degrees
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Routing:
- net Net-(D42-K): track 0.00 -> 534.9 mm, vias 0 -> 2
- net Net-(D29-K): track 0.00 -> 439.6 mm, vias 0 -> 3
- net Net-(U1-GPIO8): track 0.00 -> 425.2 mm
- net Net-(D54-K): track 0.00 -> 402.4 mm
- net GND: track 0.00 -> 347.5 mm, vias 0 -> 2
- net Net-(U1-GPIO27_ADC1): track 0.00 -> 334.5 mm, vias 0 -> 2
- net Net-(D15-K): track 0.00 -> 332.3 mm
- net Net-(U1-GPIO1): track 0.00 -> 325.8 mm
- net Net-(U1-GPIO9): track 0.00 -> 300.1 mm
- net Net-(U1-GPIO0): track 0.00 -> 289.1 mm
- net Net-(U1-GPIO28_ADC2): track 0.00 -> 287.7 mm
- net uncb: track 0.00 -> 276.9 mm, vias 0 -> 1
- net Net-(D1-K): track 0.00 -> 270.0 mm
- net Net-(U1-GPIO10): track 0.00 -> 269.3 mm
- net unca: track 0.00 -> 261.5 mm
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Other:
- board outline added: 290 x 123.5 mm
- board text added: "(symbol "LOGO" (pin_names (offset 1.016)) (in_bom yes) (on_board yes) (property "Reference" "#G" (at 0 9.10167 0) (effects (font (size 1.27 1.27)) hide) ) (property "Value" "LOGO" (at 0 -9.10167 0) (effects (font (size 1.27 1.27)) hide) ) (property "Footprint" "" (at 0 0 0) (effects (font (size 1.27 1.27)) hide) ) (property "Datasheet" "" (at 0 0 0) (effects (font (size 1.27 1.27)) hide) ) (symbo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"
- board text added: "designed by Daksh Vohra"
- board text added: "no maidens?"

Commit message: production stuff
Parts:
- added D64: LED_Small, LED_THT:LED_D5.0mm, F.Cu at (224.5, 106.2)
- added D65: LED_Small, LED_THT:LED_D5.0mm, F.Cu at (187.0, 106.2)
- added D66: LED_Small, LED_THT:LED_D5.0mm, F.Cu at (147.5, 106.2)
- added D67: LED_Small, LED_THT:LED_D5.0mm, F.Cu at (237.0, 106.2)
- added D68: LED_Small, LED_THT:LED_D5.0mm, F.Cu at (199.5, 106.2)
- added D69: LED_Small, LED_THT:LED_D5.0mm, F.Cu at (161.0, 106.2)
- added D70: LED_Small, LED_THT:LED_D5.0mm, F.Cu at (249.5, 106.2)
- added D71: LED_Small, LED_THT:LED_D5.0mm, F.Cu at (212.0, 106.2)
- added D72: LED_Small, LED_THT:LED_D5.0mm, F.Cu at (174.5, 106.2)
- added R1: 330Ω, Resistor_THT:R_Axial_DIN0309_L9.0mm_D3.2mm_P20.32mm_Horizontal, B.Cu at (140.9, 99.9)
- added R2: 330Ω, Resistor_THT:R_Axial_DIN0309_L9.0mm_D3.2mm_P20.32mm_Horizontal, B.Cu at (140.9, 104.7)
- added R3: 330Ω, Resistor_THT:R_Axial_DIN0309_L9.0mm_D3.2mm_P20.32mm_Horizontal, B.Cu at (140.9, 109.4)
- D1, D10, D11, D12, D13, D14, D15, D16, D17, D18, D19, D2, D20, D21, D22, D23, D24, D25, D26, D27, D28, D29, D3, D30, D31, D32, D33, D34, D35, D36, D37, D38, D39, D4, D40, D41, D42, D43, D44, D45, D46, D47, D48, D49, D5, D50, D51, D52, D53, D54, D55, D56, D57, D58, D59, D6, D60, D61, D62, D63, D7, D8, D9: moved to B.Cu
- U1: footprint Module:RaspberryPi_Pico_Common_THT -> pico:RPi_Pico_SMD_TH
- moved D63 112.0 mm to (343.5, 110.3)
- moved SW63 95.9 mm to (326.2, 103.7)
- moved U1 95.8 mm to (87.0, 105.4)
- moved D29 90.8 mm to (64.5, 171.5)
- moved D55 90.4 mm to (88.5, 208.7)
- moved D53 90.2 mm to (297.5, 190.3)
- moved D5 90.1 mm to (140.5, 132.5)
- moved D1 90.1 mm to (64.5, 132.5)
- moved D14 90.1 mm to (312.5, 132.3)
- moved D54 90.0 mm to (64.5, 208.7)
- moved D15 90.0 mm to (64.5, 151.5)
- moved D3 90.0 mm to (102.5, 132.3)
- moved D48 90.0 mm to (202.5, 189.7)
- moved D30 90.0 mm to (97.5, 170.5)
- moved D6 89.9 mm to (159.5, 132.5)
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Connections:
- net enca renamed re4
- net encb renamed re3
- net unca renamed re2
- net uncb renamed re1
- D1 pad 1: Net-(D1-K) -> row1
- D10 pad 1: Net-(D1-K) -> row1
- D11 pad 1: Net-(D1-K) -> row1
- D12 pad 1: Net-(D1-K) -> row1
- D13 pad 1: Net-(D1-K) -> row1
- D14 pad 1: Net-(D1-K) -> row1
- D15 pad 1: Net-(D15-K) -> row2
- D16 pad 1: Net-(D15-K) -> row2
- D17 pad 1: Net-(D15-K) -> row2
- D18 pad 1: Net-(D15-K) -> row2
- D19 pad 1: Net-(D15-K) -> row2
- D2 pad 1: Net-(D1-K) -> row1
- D20 pad 1: Net-(D15-K) -> row2
- D21 pad 1: Net-(D15-K) -> row2
- D22 pad 1: Net-(D15-K) -> row2
- D23 pad 1: Net-(D15-K) -> row2
- D24 pad 1: Net-(D15-K) -> row2
- D25 pad 1: Net-(D15-K) -> row2
- D26 pad 1: Net-(D15-K) -> row2
- D27 pad 1: Net-(D15-K) -> row2
- D28 pad 1: Net-(D15-K) -> row2
- D29 pad 1: Net-(D29-K) -> row3
- D3 pad 1: Net-(D1-K) -> row1
- D30 pad 1: Net-(D29-K) -> row3
- D31 pad 1: Net-(D29-K) -> row3
- D32 pad 1: Net-(D29-K) -> row3
- D33 pad 1: Net-(D29-K) -> row3
- D34 pad 1: Net-(D29-K) -> row3
- D35 pad 1: Net-(D29-K) -> row3
- D36 pad 1: Net-(D29-K) -> row3
- D37 pad 1: Net-(D29-K) -> row3
- D38 pad 1: Net-(D29-K) -> row3
- D39 pad 1: Net-(D29-K) -> row3
- D4 pad 1: Net-(D1-K) -> row1
- D40 pad 1: Net-(D29-K) -> row3
- D41 pad 1: Net-(D29-K) -> row3
- D42 pad 1: Net-(D42-K) -> row4
- D43 pad 1: Net-(D42-K) -> row4
- D44 pad 1: Net-(D42-K) -> row4
- D45 pad 1: Net-(D42-K) -> row4
- D46 pad 1: Net-(D42-K) -> row4
- D47 pad 1: Net-(D42-K) -> row4
- D48 pad 1: Net-(D42-K) -> row4
- D49 pad 1: Net-(D42-K) -> row4
- D5 pad 1: Net-(D1-K) -> row1
- D50 pad 1: Net-(D42-K) -> row4
- D51 pad 1: Net-(D42-K) -> row4
- D52 pad 1: Net-(D42-K) -> row4
- D53 pad 1: Net-(D42-K) -> row4
- D54 pad 1: Net-(D54-K) -> row5
- D55 pad 1: Net-(D54-K) -> row5
- D56 pad 1: Net-(D54-K) -> row5
- D57 pad 1: Net-(D54-K) -> row5
- D58 pad 1: Net-(D54-K) -> row5
- D59 pad 1: Net-(D54-K) -> row5
- D6 pad 1: Net-(D1-K) -> row1
- D60 pad 1: Net-(D54-K) -> row5
- D61 pad 1: Net-(D54-K) -> row5
- D62 pad 1: Net-(D29-K) -> row3
- D63 pad 1: Net-(D42-K) -> row4
- D7 pad 1: Net-(D1-K) -> row1
- D8 pad 1: Net-(D1-K) -> row1
- D9 pad 1: Net-(D1-K) -> row1
- SW1 pad 1: Net-(U1-GPIO15) -> col1
- SW10 pad 1: Net-(U1-GPIO6) -> col10
- SW11 pad 1: Net-(U1-GPIO0) -> col11
- SW12 pad 1: Net-(U1-GPIO1) -> col12
- SW13 pad 1: Net-(U1-GPIO28_ADC2) -> col13
- SW14 pad 1: Net-(U1-GPIO27_ADC1) -> col14
- SW15 pad 1: Net-(U1-GPIO15) -> col1
- SW16 pad 1: Net-(U1-GPIO14) -> col2
- SW17 pad 1: Net-(U1-GPIO13) -> col3
- SW18 pad 1: Net-(U1-GPIO12) -> col4
- SW19 pad 1: Net-(U1-GPIO11) -> col5
- SW2 pad 1: Net-(U1-GPIO14) -> col2
- SW20 pad 1: Net-(U1-GPIO10) -> col6
- SW21 pad 1: Net-(U1-GPIO9) -> col7
- SW22 pad 1: Net-(U1-GPIO8) -> col8
- SW23 pad 1: Net-(U1-GPIO7) -> col9
- SW24 pad 1: Net-(U1-GPIO6) -> col10
- SW25 pad 1: Net-(U1-GPIO0) -> col11
- SW26 pad 1: Net-(U1-GPIO1) -> col12
- SW27 pad 1: Net-(U1-GPIO28_ADC2) -> col13
- SW28 pad 1: Net-(U1-GPIO27_ADC1) -> col14
- SW29 pad 1: Net-(U1-GPIO15) -> col1
- SW3 pad 1: Net-(U1-GPIO13) -> col3
- SW30 pad 1: Net-(U1-GPIO14) -> col2
- SW31 pad 1: Net-(U1-GPIO13) -> col3
- SW32 pad 1: Net-(U1-GPIO12) -> col4
- SW33 pad 1: Net-(U1-GPIO11) -> col5
- SW34 pad 1: Net-(U1-GPIO10) -> col6
- SW35 pad 1: Net-(U1-GPIO9) -> col7
- SW36 pad 1: Net-(U1-GPIO8) -> col8
- SW37 pad 1: Net-(U1-GPIO7) -> col9
- SW38 pad 1: Net-(U1-GPIO6) -> col10
- SW39 pad 1: Net-(U1-GPIO0) -> col11
- SW4 pad 1: Net-(U1-GPIO12) -> col4
- SW40 pad 1: Net-(U1-GPIO1) -> col12
- SW41 pad 1: Net-(U1-GPIO28_ADC2) -> col13
- SW42 pad 1: Net-(U1-GPIO15) -> col1
- SW43 pad 1: Net-(U1-GPIO14) -> col2
- SW44 pad 1: Net-(U1-GPIO13) -> col3
- SW45 pad 1: Net-(U1-GPIO12) -> col4
- SW46 pad 1: Net-(U1-GPIO11) -> col5
- SW47 pad 1: Net-(U1-GPIO10) -> col6
- SW48 pad 1: Net-(U1-GPIO9) -> col7
- SW49 pad 1: Net-(U1-GPIO8) -> col8
- SW5 pad 1: Net-(U1-GPIO11) -> col5
- SW50 pad 1: Net-(U1-GPIO7) -> col9
- SW51 pad 1: Net-(U1-GPIO6) -> col10
- SW52 pad 1: Net-(U1-GPIO0) -> col11
- SW53 pad 1: Net-(U1-GPIO1) -> col12
- SW54 pad 1: Net-(U1-GPIO15) -> col1
- SW55 pad 1: Net-(U1-GPIO14) -> col2
- SW56 pad 1: Net-(U1-GPIO13) -> col3
- SW57 pad 1: Net-(U1-GPIO12) -> col4
- SW58 pad 1: Net-(U1-GPIO11) -> col5
- SW59 pad 1: Net-(U1-GPIO10) -> col6
- SW6 pad 1: Net-(U1-GPIO10) -> col6
- SW60 pad 1: Net-(U1-GPIO9) -> col7
- SW61 pad 1: Net-(U1-GPIO8) -> col8
- SW62 pad S2: Net-(U1-GPIO27_ADC1) -> col14
- SW63 pad S2: Net-(U1-GPIO27_ADC1) -> col14
- SW7 pad 1: Net-(U1-GPIO9) -> col7
- SW8 pad 1: Net-(U1-GPIO8) -> col8
- SW9 pad 1: Net-(U1-GPIO7) -> col9
- U1 pad 1: Net-(U1-GPIO0) -> col1
- U1 pad 10: Net-(U1-GPIO7) -> col8
- U1 pad 11: Net-(U1-GPIO8) -> col9
- U1 pad 12: Net-(U1-GPIO9) -> col10
- U1 pad 14: Net-(U1-GPIO10) -> col11
- U1 pad 15: Net-(U1-GPIO11) -> col12
- U1 pad 16: Net-(U1-GPIO12) -> col13
- U1 pad 17: Net-(U1-GPIO13) -> col14
- U1 pad 19: Net-(U1-GPIO14) -> row1
- U1 pad 2: Net-(U1-GPIO1) -> col2
- U1 pad 20: Net-(U1-GPIO15) -> row2
- U1 pad 21: unconnected-(U1-GPIO16-Pad21) -> row3
- U1 pad 22: Net-(D29-K) -> row4
- U1 pad 24: Net-(D42-K) -> row5
- U1 pad 31: Net-(D54-K) -> green_anode
- U1 pad 32: Net-(U1-GPIO27_ADC1) -> red_anode
- U1 pad 34: Net-(U1-GPIO28_ADC2) -> blue_anode
- U1 pad 4: unconnected-(U1-GPIO2-Pad4) -> col3
- U1 pad 5: unconnected-(U1-GPIO3-Pad5) -> col4
- U1 pad 6: Net-(D1-K) -> col5
- U1 pad 7: Net-(D15-K) -> col6
- U1 pad 9: Net-(U1-GPIO6) -> col7
Routing:
- net Net-(D42-K): track 534.9 -> 0.00 mm, vias 2 -> 0
- net row4: track 0.00 -> 463.8 mm, vias 0 -> 3
- net row3: track 0.00 -> 451.5 mm, vias 0 -> 1
- net Net-(D29-K): track 439.6 -> 0.00 mm, vias 3 -> 0
- net row5: track 0.00 -> 438.4 mm, vias 0 -> 5
- net Net-(U1-GPIO8): track 425.2 -> 0.00 mm
- net Net-(D54-K): track 402.4 -> 0.00 mm
- net row2: track 0.00 -> 347.3 mm
- net Net-(U1-GPIO27_ADC1): track 334.5 -> 0.00 mm, vias 2 -> 0
- net Net-(D15-K): track 332.3 -> 0.00 mm
- net col8: track 0.00 -> 329.9 mm
- net Net-(U1-GPIO1): track 325.8 -> 0.00 mm
- net col7: track 0.00 -> 311.8 mm
- net col14: track 0.00 -> 307.4 mm
- net Net-(U1-GPIO9): track 300.1 -> 0.00 mm
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Other:
- board size 290 x 123.5 mm -> 290.9 x 123.4 mm
- board text removed: "(symbol "LOGO" (pin_names (offset 1.016)) (in_bom yes) (on_board yes) (property "Reference" "#G" (at 0 9.10167 0) (effects (font (size 1.27 1.27)) hide) ) (property "Value" "LOGO" (at 0 -9.10167 0) (effects (font (size 1.27 1.27)) hide) ) (property "Footprint" "" (at 0 0 0) (effects (font (size 1.27 1.27)) hide) ) (property "Datasheet" "" (at 0 0 0) (effects (font (size 1.27 1.27)) hide) ) (symbo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"
- board text removed: "designed by Daksh Vohra"
- board text removed: "no maidens?"
